File: Shield.sch (EAGLE design)
At the start: 18 parts, among them Q8 TIP120, U2 ARDUINO_SHIELDNO_SILK

Commit message: Converted to single board
git-svn-id: svn+ssh://petrocik.net/home/svn/repo/uci_gate/branches/hardware/uci_gate/3.x@90 8c868176-b666-4d83-8e7f-acb7c29fc81a
Parts:
- removed R9: 100, SparkFun-Passives:RESISTOR1206
- added C2: 22pf, SparkFun-Capacitors:CAP1206
- added C3: 0.1uf, SparkFun-Capacitors:CAP1206
- added C6: (no value), SparkFun-Capacitors:CAPPTH1
- added C7, C8: 10uf, SparkFun-Capacitors:CAPPTH
- added J1: AVR_SPI_PRG_6PTH, SparkFun-Connectors:AVR_SPI_PRG_6PTH
- added R4: 10K, SparkFun-Passives:RESISTOR1206
- added U4: ATMEGA328P_PDIP, SparkFun-DigitalIC:ATMEGA328P_PDIP
- added Y1: 16Mhz, SparkFun-FreqCtrl:CRYSTALHC49US
- C1: value (none) -> 22pf; device SparkFun-Capacitors:CAPPTH1 -> SparkFun-Capacitors:CAP1206
- U2: value ARDUINO_SHIELDNO_SILK -> LM78XX-TO252-3; device SparkFun-Boards:ARDUINO_SHIELDNO_SILK -> element14-com:LM78XX-TO252-3
Connections:
- net N$6 renamed GATE
- removed net N$1 (its old number): U$1.B1, U2.D2
- removed net N$10: LIGHT.7, U$1.C1
- removed net N$11: U$2.SCL, U2.A5
- removed net N$13: R7.2, U2.*D9
- removed net N$14: U$2.SDA, U2.A4
- removed net N$16: BT_HDR.2, U2.RX
- removed net N$18: BT_HDR.4, R8.2, TMR.1, U$2.VCC, U2.5V
- removed net N$20: R9.1, U2.D12
- removed net N$21: R8.1, R9.2, STRT.1
- removed net N$22: R10.1, TMR.2, U2.A0
- removed net N$23: R1.1, U2.TX
- removed net N$7: LIGHT.1, U$1.C4
- removed net N$8: LIGHT.3, U$1.C3
- removed net N$9: LIGHT.5, U$1.C2
- new net 5V: BT_HDR.4, C3.2, C7.1, J1.2, R4.1, R8.2, TMR.1, U$2.VCC, U2.OUT, U4.AVCC, U4.VCC
- new net A0: R10.1, TMR.2, U4.PC0(ADC0)
- new net A4: U$2.SDA, U4.PC4(ADC4/SDA)
- new net A5: U$2.SCL, U4.PC5(ADC5/SCL)
- new net D2: U$1.B1, U4.PD2(INT0)
- new net D3: U$1.B2, U4.PD3(INT1)
- new net D4: U$1.B3, U4.PD4(XCK/T0)
- new net D5: U$1.B4, U4.PD5(T1)
- new net D6: U$1.B5, U4.PD6(AIN0)
- new net D7: R8.1, STRT.1, U4.PD7(AIN1)
- new net D9: R7.2, U4.PB1(OC1A)
- new net MISO: J1.1, U4.PB4(MISO)
- new net MOSI: J1.4, U4.PB3(MOSI/OC2)
- new net N$15: C1.2, U4.PB6(XTAL1/TOSC1), Y1.2
- new net N$24: C2.2, U4.PB7(XTAL2/TOSC2), Y1.1
- new net RESET: J1.5, R4.2, U4.PC6(/RESET)
- new net RX: BT_HDR.2, U4.PD0(RXD)
- new net SCK: J1.3, U4.PB5(SCK)
- new net TX: R1.1, U4.PD1(TXD)
- net GND: now also C1.1, C2.1, C3.1, C6.2, C7.2, C8.2, J1.6, U2.COM, U4.GND@1, U4.GND@2; no longer C1.2, U2.GND@0, U2.GND@1, U2.GND@2
- net N$2: now also LIGHT.1, U$1.C1; no longer U$1.B2, U2.*D3
- net N$3: now also LIGHT.3, U$1.C2; no longer U$1.B3, U2.D4
- net N$4: now also LIGHT.5, U$1.C3; no longer U$1.B4, U2.*D5
- net N$5: now also LIGHT.7, U$1.C4; no longer U$1.B5, U2.*D6
- net VCC: now also C6.1, C8.1, U2.IN; no longer C1.1, U2.VIN
Other:
- moved on the sheet: BT_HDR, C1, GATE, LIGHT, PWR, Q8, R1, R10, R2, R7, R8, SPKR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

Commit message: Improvement component placement
git-svn-id: svn+ssh://petrocik.net/home/svn/repo/uci_gate/branches/hardware/uci_gate/3.x@94 8c868176-b666-4d83-8e7f-acb7c29fc81a
Parts:
- C6: value (none) -> 1500uf
Changed lines of the file:
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@@
 <part name="R1" library="SparkFun-Passives" deviceset="RESISTOR" device="1206" value="1K"/>
 <part name="R2" library="SparkFun-Passives" deviceset="RESISTOR" device="1206" value="2K"/>
-<part name="C6" library="SparkFun-Capacitors" deviceset="CAP" device="PTH1"/>
+<part name="C6" library="SparkFun-Capacitors" deviceset="CAP" device="PTH1" value="1500uf"/>
 <part name="GND2" library="SparkFun-Aesthetics" deviceset="GND" device=""/>
 <part name="Y1" library="SparkFun-FreqCtrl" deviceset="CRYSTAL" device="HC49US" value="16Mhz"/>

Commit message: Fixed 12v relay voltage
git-svn-id: svn+ssh://petrocik.net/home/svn/repo/uci_gate/branches/hardware/uci_gate/3.x@133 8c868176-b666-4d83-8e7f-acb7c29fc81a
Parts:
- removed R8: 10K, SparkFun-Passives:RESISTOR1206
Connections:
- net 5V: no longer R8.2
- net D7: no longer R8.1
Changed lines of the file:
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@@
 <?xml version="1.0" encoding="utf-8"?>
 <!DOCTYPE eagle SYSTEM "eagle.dtd">
-<eagle version="6.5.0">
+<eagle version="7.2.0">
 <drawing>
 <settings>
@@
 <part name="SPKR" library="SparkFun-Connectors" deviceset="M02" device="3.5MM"/>
 <part name="Q8" library="ucigate" deviceset="TIP120" device=""/>
-<part name="R8" library="SparkFun-Passives" deviceset="RESISTOR" device="1206" value="10K"/>
 <part name="STRT" library="SparkFun-Connectors" deviceset="M02" device="3.5MM"/>
 <part name="R10" library="SparkFun-Passives" deviceset="RESISTOR" device="1206" value="10K"/>
@@
 <instance part="SPKR" gate="G$1" x="30.48" y="38.1" rot="R180"/>
 <instance part="Q8" gate="1" x="-5.08" y="30.48"/>
-<instance part="R8" gate="G$1" x="-15.24" y="114.3" rot="R180"/>
 <instance part="STRT" gate="G$1" x="12.7" y="114.3" rot="R180"/>
 <instance part="R10" gate="G$1" x="-60.96" y="-2.54"/>
@@
 <net name="D7" class="0">
 <segment>
-<pinref part="R8" gate="G$1" pin="1"/>
-<wire x1="-5.08" y1="114.3" x2="-10.16" y2="114.3" width="0.1524" layer="91"/>
 <wire x1="-5.08" y1="114.3" x2="5.08" y2="114.3" width="0.1524" layer="91"/>
-<junction x="-5.08" y="114.3"/>
 <pinref part="STRT" gate="G$1" pin="1"/>
 <wire x1="-5.08" y1="114.3" x2="-5.08" y2="109.22" width="0.1524" layer="91"/>
@@
 </segment>
 <segment>
-<pinref part="R8" gate="G$1" pin="2"/>
-<wire x1="-20.32" y1="114.3" x2="-25.4" y2="114.3" width="0.1524" layer="91"/>
-<label x="-25.4" y="114.3" size="1.27" layer="95" rot="R180" xref="yes"/>
-</segment>
-<segment>
