File: hardware/Shield.sch (EAGLE design)
At the start: 25 parts, among them J1 AVR_SPI_PRG_6PTH, Q8 TIP120, U2 LM78XX-TO252-3, U4 ATMEGA328P_PDIP, Y1 16Mhz

Commit message: Restored lost RAM board design during migration from svn
Parts:
- removed R10: 10K, SparkFun-Passives:RESISTOR1206
- added D1: (no value), SparkFun-DiscreteSemi:DIODE1N4148
- added D3: Zener, SparkFun-DiscreteSemi:DIODE-ZENER
- added Q2: MMBT5088, SparkFun-DiscreteSemi:TRANSISTOR_NPNMMBT5088
- added R3: 1K, SparkFun-Passives:RESISTOR1206
- added RELAY-JSM: RELAY-JSMJSM, petrocik:RELAY-JSMJSM
- added TMR2: (no value), SparkFun-Connectors:M023.5MM
- GATE: device SparkFun-Connectors:M023.5MM -> SparkFun-Connectors:M03-SCREW-5MM; PROD_ID (none) -> CONN-10134
- renumbered TMR to TMR1, U$1 to MC1413D, U$2 to 24AA512, U2 to LM78M05, U4 to ATMEGA328P
Connections:
- removed net GATE: GATE.2, MC1413D.C5
- new net A1: ATMEGA328P.PC1(ADC1), TMR1.2
- new net COIL: D3.C, Q2.C, RELAY-JSM.COIL2
- new net DIODENODE: D1.A, D3.A
- new net N$6: GATE.2, RELAY-JSM.MAIN
- new net N$9: Q2.B, R3.2
- new net NC: GATE.1, RELAY-JSM.NC
- new net NO: GATE.3, RELAY-JSM.NO
- net 5V: no longer TMR1.1
- net A0: now also TMR2.2; no longer R10.1, TMR1.2
- net D6: now also R3.1; no longer MC1413D.B5
- net GND: now also Q2.E, TMR1.1, TMR2.1; no longer R10.2
- net N$2: now also LIGHT.8; no longer LIGHT.1
- net N$3: now also LIGHT.4, MC1413D.C3; no longer LIGHT.3, MC1413D.C2
- net N$4: now also LIGHT.2, MC1413D.C4; no longer LIGHT.5, MC1413D.C3
- net N$5: now also LIGHT.6, MC1413D.C2; no longer LIGHT.7, MC1413D.C4
- net VCC: now also D1.C, LIGHT.1, LIGHT.3, LIGHT.5, LIGHT.7, RELAY-JSM.COIL1; no longer GATE.1, LIGHT.2, LIGHT.4, LIGHT.6, LIGHT.8
Other:
- moved on the sheet: C6, LIGHT, Q8, R7, SPKR

Commit message: 4.2
Parts:
- removed TMR1, TMR2: (no value), SparkFun-Connectors:M023.5MM
- added JP3: TMR, SparkFun-Connectors:M04SCREW
- added PMR2: TMR, SparkFun-Connectors:M023.5MM
- added R10: 10K, petrocik:RESISTOR-ARRAY
Connections:
- new net A2: ATMEGA328P.PC2(ADC2), R10D2.2, R10E.2
- new net A3: ATMEGA328P.PC3(ADC3), R10F.2, R10G.2
- new net N$11: JP3.4, R10F.1
- new net N$18: JP3.2, R10C.1
- new net N$20: JP3.3, R10D2.1
- new net N$7: JP3.1, R10A.1
- net A0: now also R10A.2, R10B.2; no longer TMR2.2
- net A1: now also R10C.2, R10D.2; no longer TMR1.2
- net GND: now also PMR2.2, R10B.1, R10D.1, R10E.1, R10G.1; no longer TMR1.1, TMR2.1
- net VCC: now also PMR2.1

Commit message: Starting 4.3 board developement
Parts:
- removed D1: (no value), SparkFun-DiscreteSemi:DIODE1N4148
- removed D3: Zener, SparkFun-DiscreteSemi:DIODE-ZENER
- removed GATE: (no value), SparkFun-Connectors:M03-SCREW-5MM
- removed JP3: TMR, SparkFun-Connectors:M04SCREW
- removed Q2: MMBT5088, SparkFun-DiscreteSemi:TRANSISTOR_NPNMMBT5088
- removed R3: 1K, SparkFun-Passives:RESISTOR1206
- removed RELAY-JSM: RELAY-JSMJSM, petrocik:RELAY-JSMJSM
- added J2: TMR, SparkFun-Connectors:CONN_04SCREW
- added J3: RELAY, SparkFun-Connectors:CONN_03SCREW
Connections:
- removed net COIL: D3.C, Q2.C, RELAY-JSM.COIL2
- removed net DIODENODE: D1.A, D3.A
- removed net N$6: GATE.2, RELAY-JSM.MAIN
- removed net N$9: Q2.B, R3.2
- removed net NC: GATE.1, RELAY-JSM.NC
- removed net NO: GATE.3, RELAY-JSM.NO
- net 5V: now also J3.1
- net D6: now also J3.3; no longer R3.1
- net GND: now also J3.2; no longer Q2.E
- net N$11: now also J2.4; no longer JP3.4
- net N$18: now also J2.2; no longer JP3.2
- net N$20: now also J2.3; no longer JP3.3
- net N$7: now also J2.1; no longer JP3.1
- net VCC: no longer D1.C, RELAY-JSM.COIL1

Commit message: Fixed positive and negative labels
Parts:
- C3: value 0.1uf -> 10uf
Changed lines of the file:
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@@
 <part name="C1" library="SparkFun-Capacitors" deviceset="CAP" device="1206" value="22pf"/>
 <part name="C2" library="SparkFun-Capacitors" deviceset="CAP" device="1206" value="22pf"/>
-<part name="C3" library="SparkFun-Capacitors" deviceset="CAP" device="1206" value="0.1uf"/>
+<part name="C3" library="SparkFun-Capacitors" deviceset="CAP" device="1206" value="10uf"/>
 <part name="GND3" library="SparkFun-Aesthetics" deviceset="GND" device=""/>
 <part name="GND5" library="SparkFun-Aesthetics" deviceset="GND" device=""/>
